File: cp2102.kicad_sch (KiCad schematic)
At the start: 4 parts, among them U301 CP2102-GMR

Commit message: update layout and schematics
Changed lines of the file:
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@@
     (date "2023-01-31")
+  )
+  (junction (at 66.04 39.37) (diameter 0) (color 0 0 0 0)
   )
   (junction (at 82.55 40.64) (diameter 0) (color 0 0 0 0)
@@
     (stroke (width 0) (type default))
   )
+  (wire (pts (xy 66.04 39.37) (xy 66.04 41.91))
+    (stroke (width 0) (type default))
+  )
   (wire (pts (xy 49.53 55.88) (xy 49.53 57.15))
     (stroke (width 0) (type default))
@@
     (stroke (width 0) (type default))
   )
-  (wire (pts (xy 66.04 36.83) (xy 66.04 41.91))
+  (wire (pts (xy 66.04 36.83) (xy 66.04 39.37))
     (stroke (width 0) (type default))
   )
@@
   )
   (wire (pts (xy 95.25 63.5) (xy 101.6 63.5))
+    (stroke (width 0) (type default))
+  )
+  (wire (pts (xy 66.04 39.37) (xy 69.85 39.37))
     (stroke (width 0) (type default))
   )
@@
         )
       )
+    )
+  )
+  (symbol (lib_id "power:PWR_FLAG") (at 69.85 39.37 0) (unit 1)
+    (in_bom yes) (on_board yes) (dnp no) (fields_autoplaced)
+    (property "Reference" "#FLG0301" (at 69.85 37.465 0)
+      (effects (font (size 1.27 1.27)) hide)
+    )
+    (property "Value" "PWR_FLAG" (at 69.85 35.56 0)
+      (effects (font (size 1.27 1.27)) hide)
+    )
+    (property "Footprint" "" (at 69.85 39.37 0)
+      (effects (font (size 1.27 1.27)) hide)
+    )
+    (property "Datasheet" "~" (at 69.85 39.37 0)
+      (effects (font (size 1.27 1.27)) hide)
+    )
+    (pin "1")
+    (instances
+      (project "arudino-clone"
+        (path "/7b2b1845-59f7-4bfa-9efc-3639d821cf70/8f8abbf0-5be8-4763-97a2-fa8e428b3e12"
+          (reference "#FLG0301") (unit 1)
+        )
+      )
+      (project "mini_arduino_clone"
+        (path "/8959ef53-e1d2-45fc-9f31-57ded4c60782/711dc556-c598-4177-8fc6-8d8d280e0435"
+          (reference "#FLG01") (unit 1)
+        )
+      )
